Commit message: Update model colors

File: humanSubject01/humanSubject01_66dof-bkp.urdf (robot description, URDF)
Before this commit: robot XSensStyleModel_template, 67 links, 66 joints
Links:
- link Head: mass 2.7144 -> 2.2392; geometry collision sphere radius=0.089005; visual sphere radius=0.089005
- link L3: mass 7.6908 -> 6.3444; geometry collision box size=0.13815 0.16323 0.085916; visual box size=0.13815 0.16323 0.085916
- link L5: mass 7.6908 -> 6.3444; geometry collision box size=0.13815 0.16323 0.095104; visual box size=0.13815 0.16323 0.095104
- link LeftFoot: mass 0.9802 -> 0.8086; geometry collision box size=0.17983 0.074775 0.078509; visual box size=0.17983 0.074775 0.078509
- link LeftForeArm: mass 1.508 -> 1.244; geometry collision cylinder length=0.22247 radius=0.019633; visual cylinder length=0.22247 radius=0.019633
- link LeftHand: mass 0.4524 -> 0.3732; geometry collision box size=0.11145 0.16718 0.039266; visual box size=0.11145 0.16718 0.039266
- link LeftLowerLeg: mass 2.7521 -> 2.2703; geometry collision cylinder length=0.40608 radius=0.037388; visual cylinder length=0.40608 radius=0.037388
- link LeftShoulder: mass 2.3374 -> 1.9282; geometry collision cylinder length=0.13047 radius=0.023574; visual cylinder length=0.13047 radius=0.023574
- link LeftToe: mass 0.1131 -> 0.0933; geometry collision box size=0.060173 0.074775 0.014191; visual box size=0.060173 0.074775 0.014191
- link LeftUpperArm: mass 2.262 -> 1.866; geometry collision cylinder length=0.26994 radius=0.029449; visual cylinder length=0.26994 radius=0.029449
- link LeftUpperLeg: mass 9.425 -> 7.775; geometry collision cylinder length=0.44898 radius=-0.0565; visual cylinder length=0.44898 radius=-0.0565
- link Neck: mass 0.9048 -> 0.7464; geometry collision cylinder length=0.089252 radius=0.014205; visual cylinder length=0.089252 radius=0.014205
- link Pelvis: mass 6.032 -> 4.976; geometry collision box size=0.13815 0.24914 0.097469; visual box size=0.13815 0.24914 0.097469
- link RightFoot: mass 0.9802 -> 0.8086; geometry collision box size=0.17983 0.074775 0.078509; visual box size=0.17983 0.074775 0.078509
- link RightForeArm: mass 1.508 -> 1.244; geometry collision cylinder length=0.22247 radius=0.019633; visual cylinder length=0.22247 radius=0.019633
- link RightHand: mass 1.1124 -> 1.0332; geometry collision box size=0.11145 0.16718 0.039266; visual box size=0.11145 0.16718 0.039266
- link RightLowerLeg: mass 2.7521 -> 2.2703; geometry collision cylinder length=0.40608 radius=0.037388; visual cylinder length=0.40608 radius=0.037388
- link RightShoulder: mass 2.3374 -> 1.9282; geometry collision cylinder length=0.13047 radius=0.023574; visual cylinder length=0.13047 radius=0.023574
- link RightToe: mass 0.1131 -> 0.0933; geometry collision box size=0.060173 0.074775 0.014191; visual box size=0.060173 0.074775 0.014191
- link RightUpperArm: mass 2.262 -> 1.866; geometry collision cylinder length=0.26994 radius=0.029449; visual cylinder length=0.26994 radius=0.029449
- link RightUpperLeg: mass 9.425 -> 7.775; geometry collision cylinder length=0.44898 radius=0.0565; visual cylinder length=0.44898 radius=0.0565
- link T12: mass 7.6908 -> 6.3444; geometry collision box size=0.13815 0.16323 0.085916; visual box size=0.13815 0.16323 0.085916
- link T8: mass 3.016 -> 2.488; geometry collision box size=0.13457 0.052626 0.11975; visual box size=0.13457 0.052626 0.11975
Joints:
- joint jC1Head_rotx: origin xyz=0.000997           0    0.096529 rpy=0 0 0 -> xyz=0.000152           0    0.089252 rpy=0 0 0
- joint jL1T12_rotx: origin xyz=0           0    0.081508 rpy=0 0 0 -> xyz=0           0    0.085916 rpy=0 0 0
- joint jL4L3_rotx: origin xyz=0.001106           0    0.090247 rpy=0 0 0 -> xyz=0.000374           0    0.095104 rpy=0 0 0
- joint jL5S1_rotx: origin xyz=-0.000609           0     0.10526 rpy=0 0 0 -> xyz=-0.000206           0    0.098478 rpy=0 0 0
- joint jLeftAnkle_rotx: origin xyz=-0.000118           0    -0.49826 rpy=0 0 0 -> xyz=0.000205           0    -0.40608 rpy=0 0 0
- joint jLeftBallFoot_rotx: origin xyz=0.15623           0   -0.066173 rpy=0 0 0 -> xyz=0.14456           0   -0.064752 rpy=0 0 0
- joint jLeftC7Shoulder_rotx: origin xyz=0    0.029722    0.065597 rpy=0 0 0 -> xyz=0    0.026313    0.067052 rpy=0 0 0
- joint jLeftElbow_rotx: origin xyz=0     0.31253           0 rpy=0 0 0 -> xyz=0     0.26994           0 rpy=0 0 0
- joint jLeftHip_rotx: origin xyz=0.000305    0.090327    0.002984 rpy=0 0 0 -> xyz=0.000103    0.081614    0.001009 rpy=0 0 0
- joint jLeftKnee_rotx: origin xyz=-9.6e-05           0    -0.46162 rpy=0 0 0 -> xyz=3.6e-05           0    -0.44898 rpy=0 0 0
- joint jLeftShoulder_rotx: origin xyz=0     0.15959           0 rpy=0 0 0 -> xyz=0     0.13047           0 rpy=0 0 0
- joint jLeftWrist_rotx: origin xyz=3.3e-05     0.25648           0 rpy=0 0 0 -> xyz=7.7e-05     0.22247           0 rpy=0 0 0
- joint jRightAnkle_rotx: origin xyz=-0.000118           0    -0.49826 rpy=0 0 0 -> xyz=0.000205           0    -0.40608 rpy=0 0 0
- joint jRightBallFoot_rotx: origin xyz=0.15623           0   -0.066173 rpy=0 0 0 -> xyz=0.14456           0   -0.064752 rpy=0 0 0
- joint jRightC7Shoulder_rotx: origin xyz=0   -0.029722    0.065597 rpy=0 0 0 -> xyz=0   -0.026313    0.067052 rpy=0 0 0
- joint jRightElbow_rotx: origin xyz=0    -0.31253           0 rpy=0 0 0 -> xyz=0    -0.26994           0 rpy=0 0 0
- joint jRightHip_rotx: origin xyz=0.000305   -0.090327    0.002984 rpy=0 0 0 -> xyz=0.000103   -0.081614    0.001009 rpy=0 0 0
- joint jRightKnee_rotx: origin xyz=-9.6e-05           0    -0.46162 rpy=0 0 0 -> xyz=3.6e-05           0    -0.44898 rpy=0 0 0
- joint jRightShoulder_rotx: origin xyz=0    -0.15959           0 rpy=0 0 0 -> xyz=0    -0.13047           0 rpy=0 0 0
- joint jRightWrist_rotx: origin xyz=3.3e-05    -0.25648           0 rpy=0 0 0 -> xyz=7.7e-05    -0.22247           0 rpy=0 0 0
- joint jT1C7_rotx: origin xyz=0           0     0.11632 rpy=0 0 0 -> xyz=0           0     0.11975 rpy=0 0 0
- joint jT9T8_rotx: origin xyz=0           0    0.081508 rpy=0 0 0 -> xyz=0           0    0.085916 rpy=0 0 0

File: humanSubject01/humanSubject01_66dof_colored.urdf (robot description, URDF)
Before this commit: robot XSensStyleModel_template, 67 links, 66 joints
Links:
- link Head: mass 2.7144 -> 2.2392; geometry collision sphere radius=0.089005; visual sphere radius=0.089005
- link L3: mass 7.6908 -> 6.3444; geometry collision box size=0.13815 0.16323 0.085916; visual box size=0.13815 0.16323 0.085916
- link L5: mass 7.6908 -> 6.3444; geometry collision box size=0.13815 0.16323 0.095104; visual box size=0.13815 0.16323 0.095104
- link LeftFoot: mass 0.9802 -> 0.8086; geometry collision box size=0.17983 0.074775 0.078509; visual box size=0.17983 0.074775 0.078509
- link LeftForeArm: mass 1.508 -> 1.244; geometry collision cylinder length=0.22247 radius=0.019633; visual cylinder length=0.22247 radius=0.019633
- link LeftHand: mass 0.4524 -> 0.3732; geometry collision box size=0.11145 0.16718 0.039266; visual box size=0.11145 0.16718 0.039266
- link LeftLowerLeg: mass 2.7521 -> 2.2703; geometry collision cylinder length=0.40608 radius=0.037388; visual cylinder length=0.40608 radius=0.037388
- link LeftShoulder: mass 2.3374 -> 1.9282; geometry collision cylinder length=0.13047 radius=0.023574; visual cylinder length=0.13047 radius=0.023574
- link LeftToe: mass 0.1131 -> 0.0933; geometry collision box size=0.060173 0.074775 0.014191; visual box size=0.060173 0.074775 0.014191
- link LeftUpperArm: mass 2.262 -> 1.866; geometry collision cylinder length=0.26994 radius=0.029449; visual cylinder length=0.26994 radius=0.029449
- link LeftUpperLeg: mass 9.425 -> 7.775; geometry collision cylinder length=0.44898 radius=-0.0565; visual cylinder length=0.44898 radius=-0.0565
- link Neck: mass 0.9048 -> 0.7464; geometry collision cylinder length=0.089252 radius=0.014205; visual cylinder length=0.089252 radius=0.014205
- link Pelvis: mass 6.032 -> 4.976; geometry collision box size=0.13815 0.24914 0.097469; visual box size=0.13815 0.24914 0.097469
- link RightFoot: mass 0.9802 -> 0.8086; geometry collision box size=0.17983 0.074775 0.078509; visual box size=0.17983 0.074775 0.078509
- link RightForeArm: mass 1.508 -> 1.244; geometry collision cylinder length=0.22247 radius=0.019633; visual cylinder length=0.22247 radius=0.019633
- link RightHand: mass 1.1124 -> 1.0332; geometry collision box size=0.11145 0.16718 0.039266; visual box size=0.11145 0.16718 0.039266
- link RightLowerLeg: mass 2.7521 -> 2.2703; geometry collision cylinder length=0.40608 radius=0.037388; visual cylinder length=0.40608 radius=0.037388
- link RightShoulder: mass 2.3374 -> 1.9282; geometry collision cylinder length=0.13047 radius=0.023574; visual cylinder length=0.13047 radius=0.023574
- link RightToe: mass 0.1131 -> 0.0933; geometry collision box size=0.060173 0.074775 0.014191; visual box size=0.060173 0.074775 0.014191
- link RightUpperArm: mass 2.262 -> 1.866; geometry collision cylinder length=0.26994 radius=0.029449; visual cylinder length=0.26994 radius=0.029449
- link RightUpperLeg: mass 9.425 -> 7.775; geometry collision cylinder length=0.44898 radius=0.0565; visual cylinder length=0.44898 radius=0.0565
- link T12: mass 7.6908 -> 6.3444; geometry collision box size=0.13815 0.16323 0.085916; visual box size=0.13815 0.16323 0.085916
- link T8: mass 3.016 -> 2.488; geometry collision box size=0.13457 0.052626 0.11975; visual box size=0.13457 0.052626 0.11975
Joints:
- joint jC1Head_rotx: origin xyz=0.000997           0    0.096529 rpy=0 0 0 -> xyz=0.000152           0    0.089252 rpy=0 0 0
- joint jL1T12_rotx: origin xyz=0           0    0.081508 rpy=0 0 0 -> xyz=0           0    0.085916 rpy=0 0 0
- joint jL4L3_rotx: origin xyz=0.001106           0    0.090247 rpy=0 0 0 -> xyz=0.000374           0    0.095104 rpy=0 0 0
- joint jL5S1_rotx: origin xyz=-0.000609           0     0.10526 rpy=0 0 0 -> xyz=-0.000206           0    0.098478 rpy=0 0 0
- joint jLeftAnkle_rotx: origin xyz=-0.000118           0    -0.49826 rpy=0 0 0 -> xyz=0.000205           0    -0.40608 rpy=0 0 0
- joint jLeftBallFoot_rotx: origin xyz=0.15623           0   -0.066173 rpy=0 0 0 -> xyz=0.14456           0   -0.064752 rpy=0 0 0
- joint jLeftC7Shoulder_rotx: origin xyz=0    0.029722    0.065597 rpy=0 0 0 -> xyz=0    0.026313    0.067052 rpy=0 0 0
- joint jLeftElbow_rotx: origin xyz=0     0.31253           0 rpy=0 0 0 -> xyz=0     0.26994           0 rpy=0 0 0
- joint jLeftHip_rotx: origin xyz=0.000305    0.090327    0.002984 rpy=0 0 0 -> xyz=0.000103    0.081614    0.001009 rpy=0 0 0
- joint jLeftKnee_rotx: origin xyz=-9.6e-05           0    -0.46162 rpy=0 0 0 -> xyz=3.6e-05           0    -0.44898 rpy=0 0 0
- joint jLeftShoulder_rotx: origin xyz=0     0.15959           0 rpy=0 0 0 -> xyz=0     0.13047           0 rpy=0 0 0
- joint jLeftWrist_rotx: origin xyz=3.3e-05     0.25648           0 rpy=0 0 0 -> xyz=7.7e-05     0.22247           0 rpy=0 0 0
- joint jRightAnkle_rotx: origin xyz=-0.000118           0    -0.49826 rpy=0 0 0 -> xyz=0.000205           0    -0.40608 rpy=0 0 0
- joint jRightBallFoot_rotx: origin xyz=0.15623           0   -0.066173 rpy=0 0 0 -> xyz=0.14456           0   -0.064752 rpy=0 0 0
- joint jRightC7Shoulder_rotx: origin xyz=0   -0.029722    0.065597 rpy=0 0 0 -> xyz=0   -0.026313    0.067052 rpy=0 0 0
- joint jRightElbow_rotx: origin xyz=0    -0.31253           0 rpy=0 0 0 -> xyz=0    -0.26994           0 rpy=0 0 0
- joint jRightHip_rotx: origin xyz=0.000305   -0.090327    0.002984 rpy=0 0 0 -> xyz=0.000103   -0.081614    0.001009 rpy=0 0 0
- joint jRightKnee_rotx: origin xyz=-9.6e-05           0    -0.46162 rpy=0 0 0 -> xyz=3.6e-05           0    -0.44898 rpy=0 0 0
- joint jRightShoulder_rotx: origin xyz=0    -0.15959           0 rpy=0 0 0 -> xyz=0    -0.13047           0 rpy=0 0 0
- joint jRightWrist_rotx: origin xyz=3.3e-05    -0.25648           0 rpy=0 0 0 -> xyz=7.7e-05    -0.22247           0 rpy=0 0 0
- joint jT1C7_rotx: origin xyz=0           0     0.11632 rpy=0 0 0 -> xyz=0           0     0.11975 rpy=0 0 0
- joint jT9T8_rotx: origin xyz=0           0    0.081508 rpy=0 0 0 -> xyz=0           0    0.085916 rpy=0 0 0
