Commit message: Bug fix: correct LeftUpperLeg link visual and collision radius to positive values #8

File: humanSubject01/humanSubject01_48dof.urdf (robot description, URDF)
Before this commit: robot XSensStyleModel_template, 49 links, 48 joints
Links:
- link LeftUpperLeg: geometry collision cylinder length=0.44898 radius=0.0565; visual cylinder length=0.44898 radius=0.0565

File: humanSubject01/humanSubject01_66dof-bkp.urdf (robot description, URDF)
Before this commit: robot XSensStyleModel_template, 67 links, 66 joints
Links:
- link LeftUpperLeg: geometry collision cylinder length=0.44898 radius=0.0565; visual cylinder length=0.44898 radius=0.0565

File: humanSubject01/humanSubject01_66dof.urdf (robot description, URDF)
Before this commit: robot XSensStyleModel_template, 67 links, 66 joints
Links:
- link LeftUpperLeg: geometry collision cylinder length=0.44898 radius=0.0565; visual cylinder length=0.44898 radius=0.0565

File: humanSubject01/humanSubject01_66dof_colored.urdf (robot description, URDF)
Before this commit: robot XSensStyleModel_template, 67 links, 66 joints
Links:
- link LeftUpperLeg: geometry collision cylinder length=0.44898 radius=0.0565; visual cylinder length=0.44898 radius=0.0565

File: humanSubject02/humanSubject02_48dof.urdf (robot description, URDF)
Before this commit: robot XSensStyleModel_template, 49 links, 48 joints
Links:
- link LeftUpperLeg: geometry collision cylinder length=0.47802 radius=0.060305; visual cylinder length=0.47802 radius=0.060305

File: humanSubject02/humanSubject02_66dof.urdf (robot description, URDF)
Before this commit: robot XSensStyleModel_template, 67 links, 66 joints
Links:
- link LeftUpperLeg: geometry collision cylinder length=0.47802 radius=0.060305; visual cylinder length=0.47802 radius=0.060305

File: humanSubject03/humanSubject03_48dof.urdf (robot description, URDF)
Before this commit: robot XSensStyleModel_template, 49 links, 48 joints
Links:
- link LeftUpperLeg: geometry collision cylinder length=0.46162 radius=0.058441; visual cylinder length=0.46162 radius=0.058441

File: humanSubject03/humanSubject03_66dof.urdf (robot description, URDF)
Before this commit: robot XSensStyleModel_template, 67 links, 66 joints
Links:
- link LeftUpperLeg: geometry collision cylinder length=0.46162 radius=0.058441; visual cylinder length=0.46162 radius=0.058441

File: humanSubject04/humanSubject04_48dof.urdf (robot description, URDF)
Before this commit: robot XSensStyleModel_template, 49 links, 48 joints
Links:
- link LeftUpperLeg: geometry collision cylinder length=0.48159 radius=0.060881; visual cylinder length=0.48159 radius=0.060881

File: humanSubject04/humanSubject04_66dof.urdf (robot description, URDF)
Before this commit: robot XSensStyleModel_template, 67 links, 66 joints
Links:
- link LeftUpperLeg: geometry collision cylinder length=0.48159 radius=0.060881; visual cylinder length=0.48159 radius=0.060881

File: humanSubject05/humanSubject05_48dof.urdf (robot description, URDF)
Before this commit: robot XSensStyleModel_template, 49 links, 48 joints
Links:
- link LeftUpperLeg: geometry collision cylinder length=0.4767 radius=0.060101; visual cylinder length=0.4767 radius=0.060101

File: humanSubject05/humanSubject05_66dof.urdf (robot description, URDF)
Before this commit: robot XSensStyleModel_template, 67 links, 66 joints
Links:
- link LeftUpperLeg: geometry collision cylinder length=0.4767 radius=0.060101; visual cylinder length=0.4767 radius=0.060101

File: humanSubject06/humanSubject06_48dof.urdf (robot description, URDF)
Before this commit: robot XSensStyleModel_template, 49 links, 48 joints
Links:
- link LeftUpperLeg: geometry collision cylinder length=0.52609 radius=0.066238; visual cylinder length=0.52609 radius=0.066238

File: humanSubject06/humanSubject06_66dof.urdf (robot description, URDF)
Before this commit: robot XSensStyleModel_template, 67 links, 66 joints
Links:
- link LeftUpperLeg: geometry collision cylinder length=0.52609 radius=0.066238; visual cylinder length=0.52609 radius=0.066238

File: humanSubject07/humanSubject07_48dof.urdf (robot description, URDF)
Before this commit: robot XSensStyleModel_template, 49 links, 48 joints
Links:
- link LeftUpperLeg: geometry collision cylinder length=0.51641 radius=0.065141; visual cylinder length=0.51641 radius=0.065141

File: humanSubject07/humanSubject07_66dof.urdf (robot description, URDF)
Before this commit: robot XSensStyleModel_template, 67 links, 66 joints
Links:
- link LeftUpperLeg: geometry collision cylinder length=0.51641 radius=0.065141; visual cylinder length=0.51641 radius=0.065141

File: humanSubject08/humanSubject08_48dof.urdf (robot description, URDF)
Before this commit: robot XSensStyleModel_template, 49 links, 48 joints
Links:
- link LeftUpperLeg: geometry collision cylinder length=0.47078 radius=0.059228; visual cylinder length=0.47078 radius=0.059228

File: humanSubject08/humanSubject08_66dof.urdf (robot description, URDF)
Before this commit: robot XSensStyleModel_template, 49 links, 48 joints
Links:
- link LeftUpperLeg: geometry collision cylinder length=0.47078 radius=0.059228; visual cylinder length=0.47078 radius=0.059228

Commit message: Correct sub01 hands

File: humanSubject01/humanSubject01_48dof.urdf (robot description, URDF)
Before this commit: robot XSensStyleModel_template, 49 links, 48 joints
Links:
- link RightHand: mass 1.0332 -> 0.3732

File: humanSubject01/humanSubject01_66dof-bkp.urdf (robot description, URDF)
Before this commit: robot XSensStyleModel_template, 67 links, 66 joints
Links:
- link RightHand: mass 1.0332 -> 0.3732

File: humanSubject01/humanSubject01_66dof.urdf (robot description, URDF)
Before this commit: robot XSensStyleModel_template, 67 links, 66 joints
Links:
- link RightHand: mass 1.0332 -> 0.3732

File: humanSubject01/humanSubject01_66dof_colored.urdf (robot description, URDF)
Before this commit: robot XSensStyleModel_template, 67 links, 66 joints
Links:
- link RightHand: mass 1.0332 -> 0.3732

Commit message: fix 48DoFs models joint constraints

File: humanSubject01/humanSubject01_48dof.urdf (robot description, URDF)
Before this commit: robot XSensStyleModel_template, 49 links, 48 joints
Joints:
- joint jLeftAnkle_rotx: limit lower=-0.610865 upper=0.785398 effort=30 velocity=1.0 -> lower=-0.785398 upper=0.610865 effort=30 velocity=1.0
- joint jRightC7Shoulder_rotx: limit lower=-0.0872665 upper=0.785398 effort=30 velocity=1.0 -> lower=-0.785398 upper=0.0872665 effort=30 velocity=1.0
- joint jRightHip_rotx: limit lower=-0.523599 upper=0.785398 effort=30 velocity=1.0 -> lower=-0.785398 upper=0.523599 effort=30 velocity=1.0

File: humanSubject02/humanSubject02_48dof.urdf (robot description, URDF)
Before this commit: robot XSensStyleModel_template, 49 links, 48 joints
Joints:
- joint jLeftAnkle_rotx: limit lower=-0.610865 upper=0.785398 effort=30 velocity=1.0 -> lower=-0.785398 upper=0.610865 effort=30 velocity=1.0
- joint jRightC7Shoulder_rotx: limit lower=-0.0872665 upper=0.785398 effort=30 velocity=1.0 -> lower=-0.785398 upper=0.0872665 effort=30 velocity=1.0
- joint jRightHip_rotx: limit lower=-0.523599 upper=0.785398 effort=30 velocity=1.0 -> lower=-0.785398 upper=0.523599 effort=30 velocity=1.0

File: humanSubject03/humanSubject03_48dof.urdf (robot description, URDF)
Before this commit: robot XSensStyleModel_template, 49 links, 48 joints
Joints:
- joint jLeftAnkle_rotx: limit lower=-0.610865 upper=0.785398 effort=30 velocity=1.0 -> lower=-0.785398 upper=0.610865 effort=30 velocity=1.0
- joint jRightC7Shoulder_rotx: limit lower=-0.0872665 upper=0.785398 effort=30 velocity=1.0 -> lower=-0.785398 upper=0.0872665 effort=30 velocity=1.0
- joint jRightHip_rotx: limit lower=-0.523599 upper=0.785398 effort=30 velocity=1.0 -> lower=-0.785398 upper=0.523599 effort=30 velocity=1.0

File: humanSubject04/humanSubject04_48dof.urdf (robot description, URDF)
Before this commit: robot XSensStyleModel_template, 49 links, 48 joints
Joints:
- joint jLeftAnkle_rotx: limit lower=-0.610865 upper=0.785398 effort=30 velocity=1.0 -> lower=-0.785398 upper=0.610865 effort=30 velocity=1.0
- joint jRightC7Shoulder_rotx: limit lower=-0.0872665 upper=0.785398 effort=30 velocity=1.0 -> lower=-0.785398 upper=0.0872665 effort=30 velocity=1.0
- joint jRightHip_rotx: limit lower=-0.523599 upper=0.785398 effort=30 velocity=1.0 -> lower=-0.785398 upper=0.523599 effort=30 velocity=1.0

File: humanSubject05/humanSubject05_48dof.urdf (robot description, URDF)
Before this commit: robot XSensStyleModel_template, 49 links, 48 joints
Joints:
- joint jLeftAnkle_rotx: limit lower=-0.610865 upper=0.785398 effort=30 velocity=1.0 -> lower=-0.785398 upper=0.610865 effort=30 velocity=1.0
- joint jRightC7Shoulder_rotx: limit lower=-0.0872665 upper=0.785398 effort=30 velocity=1.0 -> lower=-0.785398 upper=0.0872665 effort=30 velocity=1.0
- joint jRightHip_rotx: limit lower=-0.523599 upper=0.785398 effort=30 velocity=1.0 -> lower=-0.785398 upper=0.523599 effort=30 velocity=1.0

File: humanSubject06/humanSubject06_48dof.urdf (robot description, URDF)
Before this commit: robot XSensStyleModel_template, 49 links, 48 joints
Joints:
- joint jLeftAnkle_rotx: limit lower=-0.610865 upper=0.785398 effort=30 velocity=1.0 -> lower=-0.785398 upper=0.610865 effort=30 velocity=1.0
- joint jRightC7Shoulder_rotx: limit lower=-0.0872665 upper=0.785398 effort=30 velocity=1.0 -> lower=-0.785398 upper=0.0872665 effort=30 velocity=1.0
- joint jRightHip_rotx: limit lower=-0.523599 upper=0.785398 effort=30 velocity=1.0 -> lower=-0.785398 upper=0.523599 effort=30 velocity=1.0

File: humanSubject07/humanSubject07_48dof.urdf (robot description, URDF)
Before this commit: robot XSensStyleModel_template, 49 links, 48 joints
Joints:
- joint jLeftAnkle_rotx: limit lower=-0.610865 upper=0.785398 effort=30 velocity=1.0 -> lower=-0.785398 upper=0.610865 effort=30 velocity=1.0
- joint jRightC7Shoulder_rotx: limit lower=-0.0872665 upper=0.785398 effort=30 velocity=1.0 -> lower=-0.785398 upper=0.0872665 effort=30 velocity=1.0
- joint jRightHip_rotx: limit lower=-0.523599 upper=0.785398 effort=30 velocity=1.0 -> lower=-0.785398 upper=0.523599 effort=30 velocity=1.0

File: humanSubject08/humanSubject08_48dof.urdf (robot description, URDF)
Before this commit: robot XSensStyleModel_template, 49 links, 48 joints
Joints:
- joint jLeftAnkle_rotx: limit lower=-0.610865 upper=0.785398 effort=30 velocity=1.0 -> lower=-0.785398 upper=0.610865 effort=30 velocity=1.0
- joint jRightC7Shoulder_rotx: limit lower=-0.0872665 upper=0.785398 effort=30 velocity=1.0 -> lower=-0.785398 upper=0.0872665 effort=30 velocity=1.0
- joint jRightHip_rotx: limit lower=-0.523599 upper=0.785398 effort=30 velocity=1.0 -> lower=-0.785398 upper=0.523599 effort=30 velocity=1.0

File: humanSubject08/humanSubject08_66dof.urdf (robot description, URDF)
Before this commit: robot XSensStyleModel_template, 49 links, 48 joints
Joints:
- joint jLeftAnkle_rotx: limit lower=-0.610865 upper=0.785398 effort=30 velocity=1.0 -> lower=-0.785398 upper=0.610865 effort=30 velocity=1.0
- joint jRightC7Shoulder_rotx: limit lower=-0.0872665 upper=0.785398 effort=30 velocity=1.0 -> lower=-0.785398 upper=0.0872665 effort=30 velocity=1.0
- joint jRightHip_rotx: limit lower=-0.523599 upper=0.785398 effort=30 velocity=1.0 -> lower=-0.785398 upper=0.523599 effort=30 velocity=1.0

Commit message: Fix hip pitch joint limit

File: humanSubject01/humanSubject01_48dof.urdf (robot description, URDF)
Before this commit: robot XSensStyleModel_template, 49 links, 48 joints
Joints:
- joint jLeftHip_roty: limit lower=-0.261799 upper=2.0944 effort=30 velocity=1.0 -> lower=2.0944 upper=-0.261799 effort=30 velocity=1.0
- joint jRightHip_roty: limit lower=-0.261799 upper=2.0944 effort=30 velocity=1.0 -> lower=2.0944 upper=-0.261799 effort=30 velocity=1.0

File: humanSubject02/humanSubject02_48dof.urdf (robot description, URDF)
Before this commit: robot XSensStyleModel_template, 49 links, 48 joints
Joints:
- joint jLeftHip_roty: limit lower=-0.261799 upper=2.0944 effort=30 velocity=1.0 -> lower=2.0944 upper=-0.261799 effort=30 velocity=1.0
- joint jRightHip_roty: limit lower=-0.261799 upper=2.0944 effort=30 velocity=1.0 -> lower=2.0944 upper=-0.261799 effort=30 velocity=1.0

File: humanSubject03/humanSubject03_48dof.urdf (robot description, URDF)
Before this commit: robot XSensStyleModel_template, 49 links, 48 joints
Joints:
- joint jLeftHip_roty: limit lower=-0.261799 upper=2.0944 effort=30 velocity=1.0 -> lower=2.0944 upper=-0.261799 effort=30 velocity=1.0
- joint jRightHip_roty: limit lower=-0.261799 upper=2.0944 effort=30 velocity=1.0 -> lower=2.0944 upper=-0.261799 effort=30 velocity=1.0

File: humanSubject04/humanSubject04_48dof.urdf (robot description, URDF)
Before this commit: robot XSensStyleModel_template, 49 links, 48 joints
Joints:
- joint jLeftHip_roty: limit lower=-0.261799 upper=2.0944 effort=30 velocity=1.0 -> lower=2.0944 upper=-0.261799 effort=30 velocity=1.0
- joint jRightHip_roty: limit lower=-0.261799 upper=2.0944 effort=30 velocity=1.0 -> lower=2.0944 upper=-0.261799 effort=30 velocity=1.0

File: humanSubject05/humanSubject05_48dof.urdf (robot description, URDF)
Before this commit: robot XSensStyleModel_template, 49 links, 48 joints
Joints:
- joint jLeftHip_roty: limit lower=-0.261799 upper=2.0944 effort=30 velocity=1.0 -> lower=2.0944 upper=-0.261799 effort=30 velocity=1.0
- joint jRightHip_roty: limit lower=-0.261799 upper=2.0944 effort=30 velocity=1.0 -> lower=2.0944 upper=-0.261799 effort=30 velocity=1.0

File: humanSubject06/humanSubject06_48dof.urdf (robot description, URDF)
Before this commit: robot XSensStyleModel_template, 49 links, 48 joints
Joints:
- joint jLeftHip_roty: limit lower=-0.261799 upper=2.0944 effort=30 velocity=1.0 -> lower=2.0944 upper=-0.261799 effort=30 velocity=1.0
- joint jRightHip_roty: limit lower=-0.261799 upper=2.0944 effort=30 velocity=1.0 -> lower=2.0944 upper=-0.261799 effort=30 velocity=1.0

File: humanSubject07/humanSubject07_48dof.urdf (robot description, URDF)
Before this commit: robot XSensStyleModel_template, 49 links, 48 joints
Joints:
- joint jLeftHip_roty: limit lower=-0.261799 upper=2.0944 effort=30 velocity=1.0 -> lower=2.0944 upper=-0.261799 effort=30 velocity=1.0
- joint jRightHip_roty: limit lower=-0.261799 upper=2.0944 effort=30 velocity=1.0 -> lower=2.0944 upper=-0.261799 effort=30 velocity=1.0

File: humanSubject08/humanSubject08_48dof.urdf (robot description, URDF)
Before this commit: robot XSensStyleModel_template, 49 links, 48 joints
Joints:
- joint jLeftHip_roty: limit lower=-0.261799 upper=2.0944 effort=30 velocity=1.0 -> lower=2.0944 upper=-0.261799 effort=30 velocity=1.0
- joint jRightHip_roty: limit lower=-0.261799 upper=2.0944 effort=30 velocity=1.0 -> lower=2.0944 upper=-0.261799 effort=30 velocity=1.0

Commit message: Fix sign in joint limits

File: humanSubject01/humanSubject01_48dof.urdf (robot description, URDF)
Before this commit: robot XSensStyleModel_template, 49 links, 48 joints
Joints:
- joint jLeftHip_roty: limit lower=2.0944 upper=-0.261799 effort=30 velocity=1.0 -> lower=-2.0944 upper=0.261799 effort=30 velocity=1.0
- joint jRightHip_roty: limit lower=2.0944 upper=-0.261799 effort=30 velocity=1.0 -> lower=-2.0944 upper=0.261799 effort=30 velocity=1.0

File: humanSubject02/humanSubject02_48dof.urdf (robot description, URDF)
Before this commit: robot XSensStyleModel_template, 49 links, 48 joints
Joints:
- joint jLeftHip_roty: limit lower=2.0944 upper=-0.261799 effort=30 velocity=1.0 -> lower=-2.0944 upper=0.261799 effort=30 velocity=1.0
- joint jRightHip_roty: limit lower=2.0944 upper=-0.261799 effort=30 velocity=1.0 -> lower=-2.0944 upper=0.261799 effort=30 velocity=1.0

File: humanSubject03/humanSubject03_48dof.urdf (robot description, URDF)
Before this commit: robot XSensStyleModel_template, 49 links, 48 joints
Joints:
- joint jLeftHip_roty: limit lower=2.0944 upper=-0.261799 effort=30 velocity=1.0 -> lower=-2.0944 upper=0.261799 effort=30 velocity=1.0
- joint jRightHip_roty: limit lower=2.0944 upper=-0.261799 effort=30 velocity=1.0 -> lower=-2.0944 upper=0.261799 effort=30 velocity=1.0

File: humanSubject04/humanSubject04_48dof.urdf (robot description, URDF)
Before this commit: robot XSensStyleModel_template, 49 links, 48 joints
Joints:
- joint jLeftHip_roty: limit lower=2.0944 upper=-0.261799 effort=30 velocity=1.0 -> lower=-2.0944 upper=0.261799 effort=30 velocity=1.0
- joint jRightHip_roty: limit lower=2.0944 upper=-0.261799 effort=30 velocity=1.0 -> lower=-2.0944 upper=0.261799 effort=30 velocity=1.0

File: humanSubject05/humanSubject05_48dof.urdf (robot description, URDF)
Before this commit: robot XSensStyleModel_template, 49 links, 48 joints
Joints:
- joint jLeftHip_roty: limit lower=2.0944 upper=-0.261799 effort=30 velocity=1.0 -> lower=-2.0944 upper=0.261799 effort=30 velocity=1.0
- joint jRightHip_roty: limit lower=2.0944 upper=-0.261799 effort=30 velocity=1.0 -> lower=-2.0944 upper=0.261799 effort=30 velocity=1.0

File: humanSubject06/humanSubject06_48dof.urdf (robot description, URDF)
Before this commit: robot XSensStyleModel_template, 49 links, 48 joints
Joints:
- joint jLeftHip_roty: limit lower=2.0944 upper=-0.261799 effort=30 velocity=1.0 -> lower=-2.0944 upper=0.261799 effort=30 velocity=1.0
- joint jRightHip_roty: limit lower=2.0944 upper=-0.261799 effort=30 velocity=1.0 -> lower=-2.0944 upper=0.261799 effort=30 velocity=1.0

File: humanSubject07/humanSubject07_48dof.urdf (robot description, URDF)
Before this commit: robot XSensStyleModel_template, 49 links, 48 joints
Joints:
- joint jLeftHip_roty: limit lower=2.0944 upper=-0.261799 effort=30 velocity=1.0 -> lower=-2.0944 upper=0.261799 effort=30 velocity=1.0
- joint jRightHip_roty: limit lower=2.0944 upper=-0.261799 effort=30 velocity=1.0 -> lower=-2.0944 upper=0.261799 effort=30 velocity=1.0

File: humanSubject08/humanSubject08_48dof.urdf (robot description, URDF)
Before this commit: robot XSensStyleModel_template, 49 links, 48 joints
Joints:
- joint jLeftHip_roty: limit lower=2.0944 upper=-0.261799 effort=30 velocity=1.0 -> lower=-2.0944 upper=0.261799 effort=30 velocity=1.0
- joint jRightHip_roty: limit lower=2.0944 upper=-0.261799 effort=30 velocity=1.0 -> lower=-2.0944 upper=0.261799 effort=30 velocity=1.0
