Commit message: Add HandCOM to all main models

File: humanSubject01/humanSubject01_48dof.urdf (robot description, URDF)
Before this commit: robot XSensStyleModel_template, 49 links, 48 joints
Links:
- added link LeftHandCOM, mass 0.00001; visual box size=0 0 0
- added link RightHandCOM, mass 0.00001; visual box size=0 0 0
Joints:
- added joint jLeftHandCOM: type fixed, parent LeftHand, child LeftHandCOM, origin xyz=0 0.096206 0 rpy=0 0 0, axis 0 0 0
- added joint jRightHandCOM: type fixed, parent RightHand, child RightHandCOM, origin xyz=0 -0.096206 0 rpy=0 0 0, axis 0 0 0

File: humanSubject01/humanSubject01_66dof.urdf (robot description, URDF)
Before this commit: robot XSensStyleModel_template, 67 links, 66 joints
Links:
- added link LeftHandCOM, mass 0.00001; visual box size=0 0 0
- added link RightHandCOM, mass 0.00001; visual box size=0 0 0
Joints:
- added joint jLeftHandCOM: type fixed, parent LeftHand, child LeftHandCOM, origin xyz=0 0.096206 0 rpy=0 0 0, axis 0 0 0
- added joint jRightHandCOM: type fixed, parent RightHand, child RightHandCOM, origin xyz=0 -0.096206 0 rpy=0 0 0, axis 0 0 0

File: humanSubject02/humanSubject02_48dof.urdf (robot description, URDF)
Before this commit: robot XSensStyleModel_template, 49 links, 48 joints
Links:
- added link LeftHandCOM, mass 0.00001; visual box size=0 0 0
- added link RightHandCOM, mass 0.00001; visual box size=0 0 0
Joints:
- added joint jLeftHandCOM: type fixed, parent LeftHand, child LeftHandCOM, origin xyz=0 0.096206 0 rpy=0 0 0, axis 0 0 0
- added joint jRightHandCOM: type fixed, parent RightHand, child RightHandCOM, origin xyz=0 -0.096206 0 rpy=0 0 0, axis 0 0 0

File: humanSubject03/humanSubject03_48dof.urdf (robot description, URDF)
Before this commit: robot XSensStyleModel_template, 49 links, 48 joints
Links:
- added link LeftHandCOM, mass 0.00001; visual box size=0 0 0
- added link RightHandCOM, mass 0.00001; visual box size=0 0 0
Joints:
- added joint jLeftHandCOM: type fixed, parent LeftHand, child LeftHandCOM, origin xyz=0 0.096206 0 rpy=0 0 0, axis 0 0 0
- added joint jRightHandCOM: type fixed, parent RightHand, child RightHandCOM, origin xyz=0 -0.096206 0 rpy=0 0 0, axis 0 0 0

File: humanSubject04/humanSubject04_48dof.urdf (robot description, URDF)
Before this commit: robot XSensStyleModel_template, 49 links, 48 joints
Links:
- added link LeftHandCOM, mass 0.00001; visual box size=0 0 0
- added link RightHandCOM, mass 0.00001; visual box size=0 0 0
Joints:
- added joint jLeftHandCOM: type fixed, parent LeftHand, child LeftHandCOM, origin xyz=0 0.096206 0 rpy=0 0 0, axis 0 0 0
- added joint jRightHandCOM: type fixed, parent RightHand, child RightHandCOM, origin xyz=0 -0.096206 0 rpy=0 0 0, axis 0 0 0

File: humanSubject04/humanSubject04_66dof.urdf (robot description, URDF)
Before this commit: robot XSensStyleModel_template, 67 links, 66 joints
Links:
- added link LeftHandCOM, mass 0.00001; visual box size=0 0 0
- added link RightHandCOM, mass 0.00001; visual box size=0 0 0
Joints:
- added joint jLeftHandCOM: type fixed, parent LeftHand, child LeftHandCOM, origin xyz=0 0.096206 0 rpy=0 0 0, axis 0 0 0
- added joint jRightHandCOM: type fixed, parent RightHand, child RightHandCOM, origin xyz=0 -0.096206 0 rpy=0 0 0, axis 0 0 0

File: humanSubject05/humanSubject05_48dof.urdf (robot description, URDF)
Before this commit: robot XSensStyleModel_template, 49 links, 48 joints
Links:
- added link LeftHandCOM, mass 0.00001; visual box size=0 0 0
- added link RightHandCOM, mass 0.00001; visual box size=0 0 0
Joints:
- added joint jLeftHandCOM: type fixed, parent LeftHand, child LeftHandCOM, origin xyz=0 0.096206 0 rpy=0 0 0, axis 0 0 0
- added joint jRightHandCOM: type fixed, parent RightHand, child RightHandCOM, origin xyz=0 -0.096206 0 rpy=0 0 0, axis 0 0 0

File: humanSubject05/humanSubject05_66dof.urdf (robot description, URDF)
Before this commit: robot XSensStyleModel_template, 67 links, 66 joints
Links:
- added link LeftHandCOM, mass 0.00001; visual box size=0 0 0
- added link RightHandCOM, mass 0.00001; visual box size=0 0 0
Joints:
- added joint jLeftHandCOM: type fixed, parent LeftHand, child LeftHandCOM, origin xyz=0 0.096206 0 rpy=0 0 0, axis 0 0 0
- added joint jRightHandCOM: type fixed, parent RightHand, child RightHandCOM, origin xyz=0 -0.096206 0 rpy=0 0 0, axis 0 0 0

File: humanSubject06/humanSubject06_48dof.urdf (robot description, URDF)
Before this commit: robot XSensStyleModel_template, 49 links, 48 joints
Links:
- added link LeftHandCOM, mass 0.00001; visual box size=0 0 0
- added link RightHandCOM, mass 0.00001; visual box size=0 0 0
Joints:
- added joint jLeftHandCOM: type fixed, parent LeftHand, child LeftHandCOM, origin xyz=0 0.096206 0 rpy=0 0 0, axis 0 0 0
- added joint jRightHandCOM: type fixed, parent RightHand, child RightHandCOM, origin xyz=0 -0.096206 0 rpy=0 0 0, axis 0 0 0

File: humanSubject06/humanSubject06_66dof.urdf (robot description, URDF)
Before this commit: robot XSensStyleModel_template, 67 links, 66 joints
Links:
- added link LeftHandCOM, mass 0.00001; visual box size=0 0 0
- added link RightHandCOM, mass 0.00001; visual box size=0 0 0
Joints:
- added joint jLeftHandCOM: type fixed, parent LeftHand, child LeftHandCOM, origin xyz=0 0.096206 0 rpy=0 0 0, axis 0 0 0
- added joint jRightHandCOM: type fixed, parent RightHand, child RightHandCOM, origin xyz=0 -0.096206 0 rpy=0 0 0, axis 0 0 0

File: humanSubject07/humanSubject07_48dof.urdf (robot description, URDF)
Before this commit: robot XSensStyleModel_template, 49 links, 48 joints
Links:
- added link LeftHandCOM, mass 0.00001; visual box size=0 0 0
- added link RightHandCOM, mass 0.00001; visual box size=0 0 0
Joints:
- added joint jLeftHandCOM: type fixed, parent LeftHand, child LeftHandCOM, origin xyz=0 0.096206 0 rpy=0 0 0, axis 0 0 0
- added joint jRightHandCOM: type fixed, parent RightHand, child RightHandCOM, origin xyz=0 -0.096206 0 rpy=0 0 0, axis 0 0 0

File: humanSubject07/humanSubject07_66dof.urdf (robot description, URDF)
Before this commit: robot XSensStyleModel_template, 67 links, 66 joints
Links:
- added link LeftHandCOM, mass 0.00001; visual box size=0 0 0
- added link RightHandCOM, mass 0.00001; visual box size=0 0 0
Joints:
- added joint jLeftHandCOM: type fixed, parent LeftHand, child LeftHandCOM, origin xyz=0 0.096206 0 rpy=0 0 0, axis 0 0 0
- added joint jRightHandCOM: type fixed, parent RightHand, child RightHandCOM, origin xyz=0 -0.096206 0 rpy=0 0 0, axis 0 0 0

File: humanSubject08/humanSubject08_48dof.urdf (robot description, URDF)
Before this commit: robot XSensStyleModel_template, 49 links, 48 joints
Links:
- added link LeftHandCOM, mass 0.00001; visual box size=0 0 0
- added link RightHandCOM, mass 0.00001; visual box size=0 0 0
Joints:
- added joint jLeftHandCOM: type fixed, parent LeftHand, child LeftHandCOM, origin xyz=0 0.096206 0 rpy=0 0 0, axis 0 0 0
- added joint jRightHandCOM: type fixed, parent RightHand, child RightHandCOM, origin xyz=0 -0.096206 0 rpy=0 0 0, axis 0 0 0
