Commit message: Correct sub02 hands

File: humanSubject02/humanSubject02_48dof.urdf (robot description, URDF)
Before this commit: robot XSensStyleModel_template, 49 links, 48 joints
Links:
- link RightHand: mass 1.1364 -> 0.4764

File: humanSubject02/humanSubject02_66dof.urdf (robot description, URDF)
Before this commit: robot XSensStyleModel_template, 67 links, 66 joints
Links:
- link RightHand: mass 1.1364 -> 0.4764
