Commit message: Correct sub03 hands

File: humanSubject03/humanSubject03_48dof.urdf (robot description, URDF)
Before this commit: robot XSensStyleModel_template, 49 links, 48 joints
Links:
- link RightHand: mass 1.1124 -> 0.4524

File: humanSubject03/humanSubject03_66dof.urdf (robot description, URDF)
Before this commit: robot XSensStyleModel_template, 67 links, 66 joints
Links:
- link RightHand: mass 1.1124 -> 0.4524
