Commit message: Add hand com frame

File: humanSubject03/humanSubject03_66dof.urdf (robot description, URDF)
Before this commit: robot XSensStyleModel_template, 67 links, 66 joints
Links:
- added link LeftHandCOM, mass 0.00001; visual box size=0 0 0
- added link RightHandCOM, mass 0.00001; visual box size=0 0 0
Joints:
- added joint jLeftHandCOM: type fixed, parent LeftHand, child LeftHandCOM, origin xyz=0 0.096206 0 rpy=0 0 0, axis 0 0 0
- added joint jRightHandCOM: type fixed, parent RightHand, child RightHandCOM, origin xyz=0 -0.096206 0 rpy=0 0 0, axis 0 0 0
