Commit message: Correct sub04 hands

File: humanSubject04/humanSubject04_48dof.urdf (robot description, URDF)
Before this commit: robot XSensStyleModel_template, 49 links, 48 joints
Links:
- link RightHand: mass 1.0962 -> 0.4362

File: humanSubject04/humanSubject04_66dof.urdf (robot description, URDF)
Before this commit: robot XSensStyleModel_template, 67 links, 66 joints
Links:
- link RightHand: mass 1.0962 -> 0.4362
