Commit message: Correct sub05 hands

File: humanSubject05/humanSubject05_48dof.urdf (robot description, URDF)
Before this commit: robot XSensStyleModel_template, 49 links, 48 joints
Links:
- link RightHand: mass 0.99 -> 0.33

File: humanSubject05/humanSubject05_66dof.urdf (robot description, URDF)
Before this commit: robot XSensStyleModel_template, 67 links, 66 joints
Links:
- link RightHand: mass 0.99 -> 0.33
