Commit message: Correct sub06 hands

File: humanSubject06/humanSubject06_48dof.urdf (robot description, URDF)
Before this commit: robot XSensStyleModel_template, 49 links, 48 joints
Links:
- link RightHand: mass 1.0872 -> 0.4272

File: humanSubject06/humanSubject06_66dof.urdf (robot description, URDF)
Before this commit: robot XSensStyleModel_template, 67 links, 66 joints
Links:
- link RightHand: mass 1.0872 -> 0.4272
