Commit message: Correct sub07 hands

File: humanSubject07/humanSubject07_48dof.urdf (robot description, URDF)
Before this commit: robot XSensStyleModel_template, 49 links, 48 joints
Links:
- link RightHand: mass 1.1334 -> 0.4734

File: humanSubject07/humanSubject07_66dof.urdf (robot description, URDF)
Before this commit: robot XSensStyleModel_template, 67 links, 66 joints
Links:
- link RightHand: mass 1.1334 -> 0.4734
