Commit message: Correct sub08 hands

File: humanSubject08/humanSubject08_48dof.urdf (robot description, URDF)
Before this commit: robot XSensStyleModel_template, 49 links, 48 joints
Links:
- link RightHand: mass 0.9912 -> 0.3312

File: humanSubject08/humanSubject08_66dof.urdf (robot description, URDF)
Before this commit: robot XSensStyleModel_template, 49 links, 48 joints
Links:
- link RightHand: mass 0.9912 -> 0.3312
