Commit message: fixed joint limits of the meshed urdf

File: humanSubjectWithMeshes/humanSubjectWithMesh.urdf (robot description, URDF)
Before this commit: robot HumanModel, 93 links, 92 joints
Joints:
- joint jLeftShoulder_rotx: limit lower=-0.8727 upper=0.8727 effort=30.0 velocity=1.0 -> lower=-1.5708 upper=2.35619 effort=30.0 velocity=1.0
- joint jLeftShoulder_roty: limit lower=-0.8727 upper=0.8727 effort=30.0 velocity=1.0 -> lower=-1.5708 upper=1.5708 effort=30.0 velocity=1.0
- joint jLeftShoulder_rotz: limit lower=-0.8727 upper=0.8727 effort=30.0 velocity=1.0 -> lower=-3.14159 upper=0.785398 effort=30.0 velocity=1.0
- joint jRightShoulder_rotx: limit lower=-0.8727 upper=0.8727 effort=30.0 velocity=1.0 -> lower=-2.35619 upper=1.5708 effort=30.0 velocity=1.0
- joint jRightShoulder_roty: limit lower=-0.8727 upper=0.8727 effort=30.0 velocity=1.0 -> lower=-1.5708 upper=1.5708 effort=30.0 velocity=1.0
- joint jRightShoulder_rotz: limit lower=-0.8727 upper=0.8727 effort=30.0 velocity=1.0 -> lower=-0.785398 upper=3.14159 effort=30.0 velocity=1.0
